File: board.kicad_pcb (KiCad board)
At the start: 2 copper layers, 55 x 62 mm, 67 parts, among them J1 PS1 DONOR HARNESS / NOT USB, J2 RESERVED REAR SERIAL / NOT US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, J3 USB-C USB2 HRO TYPE-C-31-M-12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, Q1 2N7002 DATA OD, Q2 2N7002 ACK OD, Q3 MMBT3904 AUTO-BOOT, Q4 MMBT3904 AUTO-RESET, SW1 RESET K2-1107ST-A4SW-06, SW2 BOOT K2-1107ST-A4SW-06, U1 ESP32-WROOM-32, U2 AP63203WU-7 3.3V 2A PS1 BUCK, U3 AP2112K-3.3 USB LDO, U4 TPS2113APW POWER MUX, U5 CH340C USB-UART, U6 USBLC6-2SC6 ESD

Commit message: Release PlayBridge hardware v2.0.0
Routing:
- net GND: track 0.00 -> 175.8 mm, vias 0 -> 19
- net USB_5V: track 0.00 -> 76.5 mm, vias 0 -> 15
- net PS_3V3: track 0.00 -> 75.5 mm, vias 0 -> 14
- net USB_3V3: track 0.00 -> 34.2 mm, vias 0 -> 7
- net PS_ATT: track 32.9 -> 10.1 mm, vias 3 -> 1
- net PS_CLK: track 41.6 -> 19.6 mm, vias 3 -> 1
- net USB_DP: track 0.00 -> 22.0 mm, vias 0 -> 3
- net PS_ACK: track 37.6 -> 18.3 mm, vias 3 -> 1
- net ACK_DRIVE: track 21.4 -> 3.45 mm
- net PS_CMD: track 46.5 -> 30.0 mm
- net PS_8V_RAW: track 0.00 -> 12.1 mm, vias 0 -> 1
- net PS_8V: track 18.3 -> 30.0 mm, vias 2 -> 6
- net USB_DP_RAW: track 0.00 -> 11.6 mm, vias 0 -> 2
- net USB_DM: track 0.00 -> 10.7 mm, vias 0 -> 2
- net 3V3: track 0.00 -> 10.2 mm, vias 0 -> 9
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- added copper zone on In2.Cu, net 3V3
- added copper zone on In1.Cu, net GND
Other:
- board size 55 x 62 mm -> 56.3 x 62 mm
- copper layers 2 -> 4
