File: board.kicad_sch (KiCad schematic)
At the start: 0 parts

Commit message: Release PlayBridge hardware v2.0.0
Parts:
- added C1: 22uF 16V, PlayBridge:C_1206_3216Metric, symbol PlayBridgeAuto:AUTO_C1
- added C10: 100nF, PlayBridge:C_0603_1608Metric, symbol PlayBridgeAuto:AUTO_C10
- added C11: 1uF, PlayBridge:C_0603_1608Metric, symbol PlayBridgeAuto:AUTO_C11
- added C12: 1uF EN RESET DELAY, PlayBridge:C_0603_1608Metric, symbol PlayBridgeAuto:AUTO_C12
- added C13: 100nF 25V BST, PlayBridge:C_0603_1608Metric, symbol PlayBridgeAuto:AUTO_C13
- added C2: 22uF, PlayBridge:C_1206_3216Metric, symbol PlayBridgeAuto:AUTO_C2
- added C3: 10uF, PlayBridge:C_0805_2012Metric, symbol PlayBridgeAuto:AUTO_C3
- added C4: 100nF, PlayBridge:C_0603_1608Metric, symbol PlayBridgeAuto:AUTO_C4
- added C5: 1uF, PlayBridge:C_0603_1608Metric, symbol PlayBridgeAuto:AUTO_C5
- added C6: 4.7uF, PlayBridge:C_0805_2012Metric, symbol PlayBridgeAuto:AUTO_C6
- added C7: 100nF, PlayBridge:C_0603_1608Metric, symbol PlayBridgeAuto:AUTO_C7
- added C8: 100nF, PlayBridge:C_0603_1608Metric, symbol PlayBridgeAuto:AUTO_C8
- added C9: 22uF 6.3V BUCK OUTPUT, PlayBridge:C_0805_2012Metric, symbol PlayBridgeAuto:AUTO_C9
- added D1: STATUS GREEN, PlayBridge:LED_0603_1608Metric, symbol PlayBridgeAuto:AUTO_D1
- added D2: SMBJ12A PS1 TVS, PlayBridge:D_SMA, symbol PlayBridgeAuto:AUTO_D2
- added D3: BAT54 CMD 3V3 CLAMP, PlayBridge:D_SOD-323_SILK_CLEAN, symbol PlayBridgeAuto:AUTO_D3
- added D4: BAT54 CLK 3V3 CLAMP, PlayBridge:D_SOD-323_SILK_CLEAN, symbol PlayBridgeAuto:AUTO_D4
- added D5: BAT54 ATT 3V3 CLAMP, PlayBridge:D_SOD-323_SILK_CLEAN, symbol PlayBridgeAuto:AUTO_D5
- added F1: 750mA RESETTABLE PS1 INPUT, PlayBridge:Fuse_1206_3216Metric, symbol PlayBridgeAuto:AUTO_F1
- added J1: PS1 DONOR HARNESS / NOT USB, PlayBridge:USB3_A_Molex_48393-0003_AUTHORIZED_COPY_MODEL_V3, symbol PlayBridgeAuto:AUTO_J1
- added J2: RESERVED REAR SERIAL / NOT USB / ALL CONTACTS NC, PlayBridge:USB3_A_Molex_48393-0003_RESERVED_NOT_USB_MODEL_V3, symbol PlayBridgeAuto:AUTO_J2
- added J3: USB-C USB2 HRO TYPE-C-31-M-12 PROGRAMMING, PlayBridge:USB_C_Receptacle_HRO_TYPE-C-31-M-12_INTERIOR_FANOUT_V16_C165948_MODEL, symbol PlayBridgeAuto:AUTO_J3
- added L1: 4.7uH >=2.5A SHIELDED, PlayBridge:L_Sunlord_SWPA4030S, symbol PlayBridgeAuto:AUTO_L1
- added Q1: 2N7002 DATA OD, PlayBridge:SOT-23_SILK_CLEAN_V2, symbol PlayBridgeAuto:AUTO_Q1
- added Q2: 2N7002 ACK OD, PlayBridge:SOT-23_SILK_CLEAN_V2, symbol PlayBridgeAuto:AUTO_Q2
- added Q3: MMBT3904 AUTO-BOOT, PlayBridge:SOT-23_SILK_CLEAN_V2, symbol PlayBridgeAuto:AUTO_Q3
- added Q4: MMBT3904 AUTO-RESET, PlayBridge:SOT-23_SILK_CLEAN_V2, symbol PlayBridgeAuto:AUTO_Q4
- added R1: 1k PS CMD SERIES, PlayBridge:R_0603_1608Metric_SILK_CLEAN, symbol PlayBridgeAuto:AUTO_R1
- added R10: 100k, PlayBridge:R_0603_1608Metric_SILK_CLEAN, symbol PlayBridgeAuto:AUTO_R10
- added R11: 10k EN PULLUP, PlayBridge:R_0603_1608Metric_SILK_CLEAN, symbol PlayBridgeAuto:AUTO_R11
- added R12: 10k BOOT PULLUP, PlayBridge:R_0603_1608Metric_SILK_CLEAN, symbol PlayBridgeAuto:AUTO_R12
- added R13: 1k LED LIMIT, PlayBridge:R_0603_1608Metric_SILK_CLEAN, symbol PlayBridgeAuto:AUTO_R13
- added R14: 5.1k USB-C CC1 Rd, PlayBridge:R_0402_1005Metric_SILK_CLEAN, symbol PlayBridgeAuto:AUTO_R14
- added R15: 5.1k USB-C CC2 Rd, PlayBridge:R_0402_1005Metric_SILK_CLEAN, symbol PlayBridgeAuto:AUTO_R15
- added R16: 1k UART DIV TOP, PlayBridge:R_0603_1608Metric_SILK_CLEAN, symbol PlayBridgeAuto:AUTO_R16
- added R17: 2k UART DIV BOTTOM, PlayBridge:R_0603_1608Metric_SILK_CLEAN, symbol PlayBridgeAuto:AUTO_R17
- added R18: 10k DTR BASE, PlayBridge:R_0603_1608Metric_SILK_CLEAN, symbol PlayBridgeAuto:AUTO_R18
- added R19: 10k RTS BASE, PlayBridge:R_0603_1608Metric_SILK_CLEAN, symbol PlayBridgeAuto:AUTO_R19
- added R2: 10k, PlayBridge:R_0603_1608Metric_SILK_CLEAN, symbol PlayBridgeAuto:AUTO_R2
- added R20: 700 MUX ILIM, PlayBridge:R_0603_1608Metric_SILK_CLEAN, symbol PlayBridgeAuto:AUTO_R20
- added R21: 0R USB D+ A JOIN, PlayBridge:R_0402_1005Metric_SILK_CLEAN, symbol PlayBridgeAuto:AUTO_R21
- added R22: 0R USB D+ B JOIN, PlayBridge:R_0402_1005Metric_SILK_CLEAN, symbol PlayBridgeAuto:AUTO_R22
- added R23: 0R USB D- A JOIN, PlayBridge:R_0402_1005Metric_SILK_CLEAN, symbol PlayBridgeAuto:AUTO_R23
- added R24: 0R USB D- B JOIN, PlayBridge:R_0402_1005Metric_SILK_CLEAN, symbol PlayBridgeAuto:AUTO_R24
- added R25: 0R USB LDO ENABLE, PlayBridge:R_0402_1005Metric_SILK_CLEAN, symbol PlayBridgeAuto:AUTO_R25
- added R26: 0R USB VBUS A JOIN, PlayBridge:R_0402_1005Metric_SILK_CLEAN, symbol PlayBridgeAuto:AUTO_R26
- added R27: 0R USB VBUS B JOIN, PlayBridge:R_0402_1005Metric_SILK_CLEAN, symbol PlayBridgeAuto:AUTO_R27
- added R28: 0R USB UART SUPPLY JOIN, PlayBridge:R_0402_1005Metric_SILK_CLEAN, symbol PlayBridgeAuto:AUTO_R28
- added R3: 1k PS CLK SERIES, PlayBridge:R_0603_1608Metric_SILK_CLEAN, symbol PlayBridgeAuto:AUTO_R3
- added R4: 10k, PlayBridge:R_0603_1608Metric_SILK_CLEAN, symbol PlayBridgeAuto:AUTO_R4
- added R5: 1k PS ATT SERIES, PlayBridge:R_0603_1608Metric_SILK_CLEAN, symbol PlayBridgeAuto:AUTO_R5
- added R6: 10k, PlayBridge:R_0603_1608Metric_SILK_CLEAN, symbol PlayBridgeAuto:AUTO_R6
- added R7: 100, PlayBridge:R_0603_1608Metric_SILK_CLEAN, symbol PlayBridgeAuto:AUTO_R7
- added R8: 100k, PlayBridge:R_0603_1608Metric_SILK_CLEAN, symbol PlayBridgeAuto:AUTO_R8
- added R9: 100, PlayBridge:R_0603_1608Metric_SILK_CLEAN, symbol PlayBridgeAuto:AUTO_R9
- added SW1: RESET K2-1107ST-A4SW-06, PlayBridge:SW_SPST_HRO_K2-1107ST-A4SW-06_RESET_V8, symbol PlayBridgeAuto:AUTO_SW1
- added SW2: BOOT K2-1107ST-A4SW-06, PlayBridge:SW_SPST_HRO_K2-1107ST-A4SW-06_BOOT_V8, symbol PlayBridgeAuto:AUTO_SW2
- added TP1: 3V3 TEST, PlayBridge:TestPoint_Pad_D1.5mm_SILK_CLEAN, symbol PlayBridgeAuto:AUTO_TP1
- added TP2: GND TEST, PlayBridge:TestPoint_Pad_D1.5mm_SILK_CLEAN, symbol PlayBridgeAuto:AUTO_TP2
- added TP3: UART TX TEST, PlayBridge:TestPoint_Pad_D1.5mm_SILK_CLEAN, symbol PlayBridgeAuto:AUTO_TP3
- added TP4: UART RX TEST, PlayBridge:TestPoint_Pad_D1.5mm_SILK_CLEAN, symbol PlayBridgeAuto:AUTO_TP4
- added U1: ESP32-WROOM-32, PlayBridge:ESP32-WROOM-32_D0.3mm_SILK_CLEAN, symbol PlayBridgeAuto:AUTO_U1
- added U2: AP63203WU-7 3.3V 2A PS1 BUCK, PlayBridge:TSOT-23-6, symbol PlayBridgeAuto:AUTO_U2
- added U3: AP2112K-3.3 USB LDO, PlayBridge:SOT-23-5, symbol PlayBridgeAuto:AUTO_U3
- added U4: TPS2113APW POWER MUX, PlayBridge:TSSOP-8_3x3mm_P0.65mm_AUTHORIZED_KICAD_COPY, symbol PlayBridgeAuto:AUTO_U4
- added U5: CH340C USB-UART, PlayBridge:SOIC-16_3.9x9.9mm_P1.27mm_SILK_CLEAN, symbol PlayBridgeAuto:AUTO_U5
- added U6: USBLC6-2SC6 ESD, PlayBridge:SOT-23-6, symbol PlayBridgeAuto:AUTO_U6
Connections:
- new net 3V3: C11.1 (3V3), C3.1 (3V3), C4.1 (3V3), R11.1 (3V3), R12.1 (3V3), R13.1 (3V3), TP1.1 (3V3), U1.2 (3V3), U4.7 (3V3)
- new net ACK_DRIVE: Q2.1 (ACK_DRIVE), R10.1 (ACK_DRIVE), R9.2 (ACK_DRIVE)
- new net ACK_GATE: R9.1 (ACK_GATE), U1.33 (ACK_GATE)
- new net ATT_IN: D5.2 (ATT_IN), R5.2 (ATT_IN), R6.1 (ATT_IN), U1.6 (ATT_IN)
- new net AUTO_BOOT: Q3.1 (AUTO_BOOT), R18.2 (AUTO_BOOT)
- new net AUTO_RESET: Q4.1 (AUTO_RESET), R19.2 (AUTO_RESET)
- new net BOOT: Q3.3 (BOOT), R12.2 (BOOT), SW2.1 (BOOT), U1.25 (BOOT)
- new net BUCK_BST: C13.2 (BUCK_BST), U2.6 (BUCK_BST)
- new net BUCK_SW: C13.1 (BUCK_SW), L1.1 (BUCK_SW), U2.5 (BUCK_SW)
- new net CH340_V3: C8.1 (CH340_V3), U5.4 (CH340_V3)
- new net CH_TX_5V: R16.1 (CH_TX_5V), U5.2 (CH_TX_5V)
- new net CLK_IN: D4.2 (CLK_IN), R3.2 (CLK_IN), R4.1 (CLK_IN), U1.9 (CLK_IN)
- new net CMD_IN: D3.2 (CMD_IN), R1.2 (CMD_IN), R2.1 (CMD_IN), U1.8 (CMD_IN)
- new net DATA_DRIVE: Q1.1 (DATA_DRIVE), R7.2 (DATA_DRIVE), R8.1 (DATA_DRIVE)
- new net DATA_GATE: R7.1 (DATA_GATE), U1.31 (DATA_GATE)
- new net EN: C12.1 (EN), Q4.3 (EN), R11.2 (EN), SW1.1 (EN), U1.3 (EN)
- new net GND: C1.2 (GND), C10.2 (GND), C11.2 (GND), C12.2 (GND), C2.2 (GND), C3.2 (GND), C4.2 (GND), C5.2 (GND), C6.2 (GND), C7.2 (GND), C8.2 (GND), C9.2 (GND), D2.2 (GND), J1.4 (GND), J3.A12_B1 (GND), J3.A1_B12 (GND), J3.S1 (GND), Q1.2 (GND), Q2.2 (GND), R10.2 (GND), R14.2 (GND), R15.2 (GND), R17.2 (GND), R2.2 (GND), R20.2 (GND), R4.2 (GND), R6.2 (GND), R8.2 (GND), SW1.2 (GND), SW2.2 (GND), TP2.1 (GND), U1.1 (GND), U1.15 (GND), U1.38 (GND), U1.39 (GND), U2.4 (GND), U3.2 (GND), U4.2 (GND), U4.5 (GND), U5.1 (GND), U5.15 (GND), U6.2 (GND)
- new net LED_A: D1.1 (LED_A), R13.2 (LED_A)
- new net MUX_ILIM: R20.1 (MUX_ILIM), U4.4 (MUX_ILIM)
- new net PS_3V3: C2.1 (PS_3V3), C9.1 (PS_3V3), D3.1 (PS_3V3), D4.1 (PS_3V3), D5.1 (PS_3V3), L1.2 (PS_3V3), U2.1 (PS_3V3), U4.3 (PS_3V3), U4.8 (PS_3V3)
- new net PS_8V: C1.1 (PS_8V), D2.1 (PS_8V), F1.2 (PS_8V), U2.2 (PS_8V), U2.3 (PS_8V)
- new net PS_8V_RAW: F1.1 (PS_8V_RAW), J1.8 (PS_8V_RAW)
- new net PS_ACK: J1.7 (PS_ACK), Q2.3 (PS_ACK)
- new net PS_ATT: J1.5 (PS_ATT), R5.1 (PS_ATT)
- new net PS_CLK: J1.3 (PS_CLK), R3.1 (PS_CLK)
- new net PS_CMD: J1.2 (PS_CMD), R1.1 (PS_CMD)
- new net PS_DATA: J1.6 (PS_DATA), Q1.3 (PS_DATA)
- new net STATUS_LED: D1.2 (STATUS_LED), U1.26 (STATUS_LED)
- new net UART_RX: R16.2 (UART_RX), R17.1 (UART_RX), TP4.1 (UART_RX), U1.34 (UART_RX)
- new net UART_TX: TP3.1 (UART_TX), U1.35 (UART_TX), U5.3 (UART_TX)
- new net USB_3V3: C10.1 (USB_3V3), C6.1 (USB_3V3), U3.5 (USB_3V3), U4.6 (USB_3V3)
- new net USB_5V: C5.1 (USB_5V), C7.1 (USB_5V), R25.1 (USB_5V), R26.2 (USB_5V), R27.2 (USB_5V), R28.1 (USB_5V), U3.1 (USB_5V), U6.5 (USB_5V)
- new net USB_CC1: J3.A5 (USB_CC1), R14.1 (USB_CC1)
- new net USB_CC2: J3.B5 (USB_CC2), R15.1 (USB_CC2)
- new net USB_DM: U5.6 (USB_DM), U6.6 (USB_DM)
- new net USB_DM_A: J3.A7 (USB_DM_A), R23.1 (USB_DM_A)
- new net USB_DM_B: J3.B7 (USB_DM_B), R24.1 (USB_DM_B)
- new net USB_DM_RAW: R23.2 (USB_DM_RAW), R24.2 (USB_DM_RAW), U6.1 (USB_DM_RAW)
- new net USB_DP: U5.5 (USB_DP), U6.4 (USB_DP)
- new net USB_DP_A: J3.A6 (USB_DP_A), R21.1 (USB_DP_A)
- new net USB_DP_B: J3.B6 (USB_DP_B), R22.1 (USB_DP_B)
- new net USB_DP_RAW: R21.2 (USB_DP_RAW), R22.2 (USB_DP_RAW), U6.3 (USB_DP_RAW)
- new net USB_DTR: Q4.2 (USB_DTR), R18.1 (USB_DTR), U5.13 (USB_DTR)
- new net USB_LDO_EN: R25.2 (USB_LDO_EN), U3.3 (USB_LDO_EN)
- new net USB_RTS: Q3.2 (USB_RTS), R19.1 (USB_RTS), U5.14 (USB_RTS)
- new net USB_UART_5V: R28.2 (USB_UART_5V), U5.16 (USB_UART_5V)
- new net USB_VBUS_A: J3.A4_B9 (USB_VBUS_A), R26.1 (USB_VBUS_A)
- new net USB_VBUS_B: J3.A9_B4 (USB_VBUS_B), R27.1 (USB_VBUS_B)
