File: versions/v3.0-ps1-serial-harness/board.kicad_pcb (KiCad board)
At the start: 4 copper layers, 56.3 x 62 mm, 69 parts, among them J1 PS1 DONOR HARNESS / NOT USB, J2 RESERVED REAR SERIAL / NOT US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, J3 USB-C USB2 HRO TYPE-C-31-M-12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, Q1 2N7002 DATA OD, Q2 2N7002 ACK OD, Q3 MMBT3904 AUTO-BOOT, Q4 MMBT3904 AUTO-RESET, SW1 RESET K2-1107ST-A4SW-06, SW2 BOOT K2-1107ST-A4SW-06, U1 ESP32-WROOM-32, U2 AP63203WU-7 3.3V 2A PS1 BUCK, U3 AP2112K-3.3 USB LDO, U4 TPS2113APW POWER MUX, U5 CH340C USB-UART, U6 USBLC6-2SC6 ESD

Commit message: Route J2 on dedicated ESP32 UART2 pins
Parts:
- added R30: 1k U2TX SERIES / BENCH CONFIG, PlayBridge:R_0603_1608Metric_SILK_CLEAN, F.Cu at (0.00, 0.00)
- added R31: 1k U2RX SERIES / BENCH CONFIG, PlayBridge:R_0603_1608Metric_SILK_CLEAN, F.Cu at (0.00, 0.00)
- J2: value RESERVED REAR SERIAL / NOT USB / ALL CONTACTS NC -> PS1 SERIAL / NOT USB / 3-SIGNAL CANDIDATE; footprint PlayBridge:USB3_A_Molex_48393-0003_RESERVED_NOT_USB_MODEL_V3 -> PlayBridge:USB3_A_Molex_48393-0003_PS1_SERIAL_NOT_USB_MODEL_V3
Connections:
- J2 pad 1: (no net) -> PS1_RXD
- J2 pad 4: (no net) -> PS1_TXD
- J2 pad 7: (no net) -> GND
- U1 pad 27: (no net) -> U2_RX_RAW
- U1 pad 28: (no net) -> U2_TX_RAW
Routing:
- net U2_RX_RAW: track 0.00 -> 103.3 mm, vias 0 -> 2
- net U2_TX_RAW: track 0.00 -> 93.5 mm, vias 0 -> 2
- net PS1_TXD: track 0.00 -> 22.7 mm, vias 0 -> 1
- net PS1_RXD: track 0.00 -> 22.0 mm
