File: versions/v3.0-ps1-serial-harness/board.kicad_sch (KiCad schematic)
At the start: 69 parts, among them J1 PS1 DONOR HARNESS / NOT USB, J2 RESERVED REAR SERIAL / NOT US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, J3 USB-C USB2 HRO TYPE-C-31-M-12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, Q1 2N7002 DATA OD, Q2 2N7002 ACK OD, Q3 MMBT3904 AUTO-BOOT, Q4 MMBT3904 AUTO-RESET, SW1 RESET K2-1107ST-A4SW-06, SW2 BOOT K2-1107ST-A4SW-06, U1 ESP32-WROOM-32, U2 AP63203WU-7 3.3V 2A PS1 BUCK, U3 AP2112K-3.3 USB LDO, U4 TPS2113APW POWER MUX, U5 CH340C USB-UART, U6 USBLC6-2SC6 ESD

Commit message: Route J2 on dedicated ESP32 UART2 pins
Parts:
- added R30: 1k U2TX SERIES / BENCH CONFIG, PlayBridge:R_0603_1608Metric_SILK_CLEAN, symbol Device:R
- added R31: 1k U2RX SERIES / BENCH CONFIG, PlayBridge:R_0603_1608Metric_SILK_CLEAN, symbol Device:R
- J2: value RESERVED REAR SERIAL / NOT USB / ALL CONTACTS NC -> PS1 SERIAL / NOT USB / 3-SIGNAL CANDIDATE; footprint PlayBridge:USB3_A_Molex_48393-0003_RESERVED_NOT_USB_MODEL_V3 -> PlayBridge:USB3_A_Molex_48393-0003_PS1_SERIAL_NOT_USB_MODEL_V3; Pinout RESERVED: contacts 1 through 9 and shell pads SH intentiona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 -> SONY REAR SERIAL NUMBERING PRESERVED: 1=PS1_RXD from ESP32 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; Safety NOT USB. Do not populate a harness until the PS1 rear seria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 -> NOT USB. Three-signal bench candidate only. PS1 3.5V on con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
Connections:
- net GND: now also J2.7 (GND)
- new net PS1_RXD: J2.1 (PS1_RXD), R30.2
- new net PS1_TXD: J2.4 (PS1_TXD), R31.1
- new net U2_RX_RAW: R31.2, U1.27 (U2_RX_RAW)
- new net U2_TX_RAW: R30.1, U1.28 (U2_TX_RAW)

Commit message: Record V3 PoC evidence and refresh manufacturing files
Parts:
- J2: Safety NOT USB. Three-signal bench candidate only. PS1 3.5V on con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 -> NOT USB. Three-signal PS1 serial harness validated by the u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
Changed lines of the file:
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@@
 			)
 		)
-		(property "Safety" "NOT USB. Three-signal bench candidate only. PS1 3.5V on contact 2 is intentionally isolated and must never connect to board 3V3. Logic-level compatibility is not yet verified. Full PS1 serial handshaking is not implemented."
+		(property "Safety" "NOT USB. Three-signal PS1 serial harness validated by the user/team on the documented bench PoC. PS1 3.5V on contact 2 is intentionally isolated and must never connect to board 3V3. Validation applies only to the tested hardware/protocol configuration; full PS1 serial handshaking is not implemented."
 			(at 66.04 86.36 0)
 			(hide yes)

Commit message: Replace USB-A connectors with stocked C7501856
Parts:
- J1: footprint PlayBridge:USB3_A_Molex_48393-0003_AUTHORIZED_COPY_MODEL_V3 -> PlayBridge:USB3_A_HongCheng_HC-USB3.0-L168-ZP_C7501856_PS1_FRONT_MODEL_V3; Footprint Provenance Project-local authorized geometry copy of bundled KiCad Con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 -> Official JLCPCB/EasyEDA C7501856 land geometry for Hong Che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; JLCPCB Part URL https://jlcpcb.com/partdetail/C3197928 -> https://jlcpcb.com/partdetail/HongCheng-HC_USB3_0_L168ZP/C7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; JLCPCB/LCSC Part C3197928 -> C7501856; LCSC C3197928 -> C7501856; MPN 48393-0003 -> HC-USB3.0-L168-ZP; Manufacturer Molex -> Hong Cheng; Normalized Manufacturer Number 483930003 -> HC-USB3.0-L168-ZP; Orientation Right-angle top-mount receptacle at enclosure edge; mating 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 -> Right-angle top-mount receptacle at the lower board edge; m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; Procurement Status JLCPCB selection retained; verify order-time stock -> JLCPCB in-stock assembly part; recheck live stock at order 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
- J2: footprint PlayBridge:USB3_A_Molex_48393-0003_PS1_SERIAL_NOT_USB_MODEL_V3 -> PlayBridge:USB3_A_HongCheng_HC-USB3.0-L168-ZP_C7501856_PS1_SERIAL_MODEL_V3; JLCPCB Part URL https://jlcpcb.com/partdetail/C3197928 -> https://jlcpcb.com/partdetail/HongCheng-HC_USB3_0_L168ZP/C7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; JLCPCB/LCSC Part C3197928 -> C7501856; LCSC C3197928 -> C7501856; MPN 48393-0003 -> HC-USB3.0-L168-ZP; Manufacturer Molex -> Hong Cheng; Normalized Manufacturer Number 483930003 -> HC-USB3.0-L168-ZP; Procurement Status JLCPCB selection retained; verify order-time stock -> JLCPCB in-stock assembly part; recheck live stock at order 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
Changed lines of the file:
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@@
 			)
 		)
-		(property "Footprint" "PlayBridge:USB3_A_Molex_48393-0003_AUTHORIZED_COPY_MODEL_V3"
+		(property "Footprint" "PlayBridge:USB3_A_HongCheng_HC-USB3.0-L168-ZP_C7501856_PS1_FRONT_MODEL_V3"
 			(at 30.48 86.36 0)
 			(hide yes)
@@
 			)
 		)
-		(property "Datasheet" "https://www.molex.com/en-us/products/part-detail/483930003"
+		(property "Datasheet" "https://jlcpcb.com/partdetail/HongCheng-HC_USB3_0_L168ZP/C7501856"
 			(at 30.48 86.36 0)
 			(hide yes)
@@
 			)
 		)
-		(property "Manufacturer" "Molex"
+		(property "Manufacturer" "Hong Cheng"
 			(at 30.48 86.36 0)
 			(hide yes)
@@
 			)
 		)
-		(property "MPN" "48393-0003"
+		(property "MPN" "HC-USB3.0-L168-ZP"
 			(at 30.48 86.36 0)
 			(hide yes)
@@
 			)
 		)
-		(property "Normalized Manufacturer Number" "483930003"
+		(property "Normalized Manufacturer Number" "HC-USB3.0-L168-ZP"
 			(at 30.48 86.36 0)
 			(hide yes)
@@
 			)
 		)
-		(property "JLCPCB/LCSC Part" "C3197928"
+		(property "JLCPCB/LCSC Part" "C7501856"
 			(at 30.48 86.36 0)
 			(hide yes)
@@
 			)
 		)
-		(property "Footprint Provenance" "Project-local authorized geometry copy of bundled KiCad Connector_USB:USB3_A_Molex_48393-001; land geometry references Molex drawing 483930003_sd.pdf."
+		(property "Footprint Provenance" "Official JLCPCB/EasyEDA C7501856 land geometry for Hong Cheng HC-USB3.0-L168-ZP, converted locally with easyeda2kicad."
 			(at 30.48 86.36 0)
 			(hide yes)
@@
 			)
 		)
-		(property "Orientation" "Right-angle top-mount receptacle at enclosure edge; mating mouth faces outward. PCB solder-side contact numbering is not a mating-view map: verify mirror orientation against the Molex drawing before harness assembly."
+		(property "Orientation" "Right-angle top-mount receptacle at the lower board edge; mating mouth faces outward. Signal-pad coordinates are preserved from the validated board routing."
 			(at 30.48 86.36 0)
 			(hide yes)
@@
 			)
 		)
-		(property "LCSC" "C3197928"
+		(property "LCSC" "C7501856"
 			(at 30.48 86.36 0)
 			(hide yes)
@@
 			)
 		)
-		(property "Procurement Status" "JLCPCB selection retained; verify order-time stock"
+		(property "Procurement Status" "JLCPCB in-stock assembly part; recheck live stock at order time"
 			(at 30.48 86.36 0)
 			(hide yes)
@@
 			)
 		)
-		(property "JLCPCB Part URL" "https://jlcpcb.com/partdetail/C3197928"
+		(property "JLCPCB Part URL" "https://jlcpcb.com/partdetail/HongCheng-HC_USB3_0_L168ZP/C7501856"
 			(at 30.48 86.36 0)
 			(hide yes)
@@
 			)
 		)
-		(property "Footprint" "PlayBridge:USB3_A_Molex_48393-0003_PS1_SERIAL_NOT_USB_MODEL_V3"
+		(property "Footprint" "PlayBridge:USB3_A_HongCheng_HC-USB3.0-L168-ZP_C7501856_PS1_SERIAL_MODEL_V3"
 			(at 66.04 86.36 0)
 			(hide yes)
@@
 			)
 		)
-		(property "Datasheet" "https://www.molex.com/en-us/products/part-detail/483930003"
+		(property "Datasheet" "https://jlcpcb.com/partdetail/HongCheng-HC_USB3_0_L168ZP/C7501856"
 			(at 66.04 86.36 0)
 			(hide yes)
@@
 			)
 		)
-		(property "Manufacturer" "Molex"
+		(property "Manufacturer" "Hong Cheng"
 			(at 66.04 86.36 0)
 			(hide yes)
@@
 			)
 		)
-		(property "MPN" "48393-0003"
+		(property "MPN" "HC-USB3.0-L168-ZP"
 			(at 66.04 86.36 0)
 			(hide yes)
@@
 			)
 		)
-		(property "Normalized Manufacturer Number" "483930003"
+		(property "Normalized Manufacturer Number" "HC-USB3.0-L168-ZP"
 			(at 66.04 86.36 0)
 			(hide yes)
@@
 			)
 		)
-		(property "JLCPCB/LCSC Part" "C3197928"
+		(property "JLCPCB/LCSC Part" "C7501856"
 			(at 66.04 86.36 0)
 			(hide yes)
@@
 			)
 		)
-		(property "LCSC" "C3197928"
+		(property "LCSC" "C7501856"
 			(at 66.04 86.36 0)
 			(hide yes)
@@
 			)
 		)
-		(property "Procurement Status" "JLCPCB selection retained; verify order-time stock"
+		(property "Procurement Status" "JLCPCB in-stock assembly part; recheck live stock at order time"
 			(at 66.04 86.36 0)
 			(hide yes)
@@
 			)
 		)
-		(property "JLCPCB Part URL" "https://jlcpcb.com/partdetail/C3197928"
+		(property "JLCPCB Part URL" "https://jlcpcb.com/partdetail/HongCheng-HC_USB3_0_L168ZP/C7501856"
 			(at 66.04 86.36 0)
 			(hide yes)

Commit message: Use stocked JLCPCB assembly parts
Parts:
- C1, C10, C11, C12, C13, C2, C4, C5, C6, C7, C8, D2, D3, D4, D5, F1, Q1, Q2, Q3, Q4, R1, R10, R11, R12, R13, R14, R15, R16, R17, R18, R19, R2, R21, R22, R23, R24, R25, R26, R27, R28, R3, R4, R5, R6, R7, R8, R9, U1, U2, U3, U4, U5, U6: Procurement Status JLCPCB in-stock selection verified 2026-09-22 -> JLCPCB sourcing selection verified 2026-09-25
- C3: JLCPCB Part URL https://jlcpcb.com/partdetail/C380332 -> https://jlcpcb.com/partdetail/C1713; JLCPCB/LCSC Part C380332 -> C1713; LCSC C380332 -> C1713; MPN TCC0805X5R106K160FT -> CL21A106KOQNNNE; Manufacturer CCTC -> Samsung Electro-Mechanics; Procurement Status JLCPCB in-stock selection verified 2026-09-22 -> JLCPCB sourcing selection verified 2026-09-25
- C9: JLCPCB Part URL https://jlcpcb.com/partdetail/C466795 -> https://jlcpcb.com/partdetail/C5674; JLCPCB/LCSC Part C466795 -> C5674; LCSC C466795 -> C5674; MPN C0805X5R226M6R3NT -> CL21A226MQQNNNE; Manufacturer SANYEAR -> Samsung Electro-Mechanics; Procurement Status JLCPCB in-stock selection verified 2026-09-22 -> JLCPCB sourcing selection verified 2026-09-25
- D1: value STATUS GREEN -> STATUS YELLOW-GREEN; JLCPCB Part URL https://jlcpcb.com/partdetail/C72043 -> https://jlcpcb.com/partdetail/C2289; JLCPCB/LCSC Part C72043 -> C2289; LCSC C72043 -> C2289; MPN 19-217/GHC-YR1S2/3T -> KT-0603YG; Manufacturer Everlight Electronics -> KENTO; Package 0603 green LED -> 0603 yellow-green LED; Procurement Status JLCPCB in-stock selection verified 2026-09-22 -> JLCPCB sourcing selection verified 2026-09-25
- J1: Package (none) -> USB 3.0 Type-A right-angle through-hole receptacle, 9 signa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; Procurement Status JLCPCB in-stock assembly part; recheck live stock at order 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 -> JLCPCB in-stock assembly part verified 2026-09-25; recheck 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
- J2: Footprint Provenance (none) -> Official JLCPCB/EasyEDA C7501856 land geometry for Hong Che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; Orientation (none) -> Right-angle top-mount receptacle at the lower board edge; m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; Package (none) -> USB 3.0 Type-A right-angle through-hole receptacle, 9 signa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; Procurement Status JLCPCB in-stock assembly part; recheck live stock at order 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 -> JLCPCB in-stock assembly part verified 2026-09-25; recheck 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
- L1: value 4.7uH >=2.5A SHIELDED -> 4.7uH 2.85A SHIELDED WPN4020H; footprint PlayBridge:L_Sunlord_SWPA4030S -> PlayBridge:L_Sunlord_WPN4020H; Footprint Provenance (none) -> Official Sunlord WPN4020H land pattern: 1.9mm pad gap, 1.1x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; JLCPCB Part URL https://jlcpcb.com/partdetail/C49449313 -> https://jlcpcb.com/partdetail/C98363; JLCPCB/LCSC Part C49449313 -> C98363; LCSC C49449313 -> C98363; MPN MCNR4030AF-4R7M -> WPN4020H4R7MT; Manufacturer MYX -> Sunlord; Package SMD 4.0x4.0mm, 4.7uH, 2.5A rated, 3A saturation -> SMD 4.0x4.0x2.0mm, 4.7uH +/-20%, 2.85A rated, 4.9A saturati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; Procurement Status JLCPCB in-stock selection verified 2026-09-22 -> JLCPCB sourcing selection verified 2026-09-25
- R20: value 700 MUX ILIM -> 680R MUX ILIM; Engineering Note 698R is the stocked E96 substitute for 700R; TPS2113A curre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 -> Relative to the existing 698R selection, the calculated TPS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; JLCPCB Part URL https://jlcpcb.com/partdetail/C912219 -> https://jlcpcb.com/partdetail/C23228; JLCPCB/LCSC Part C912219 -> C23228; LCSC C912219 -> C23228; MPN RMS06FT6980 -> 0603WAF6800T5E; Manufacturer TA-I -> UNI-ROYAL; Package 0603, 698R, +/-1% (700R nominal ILIM; -0.29% substitution) -> 0603, 680R, +/-1%; Procurement Status JLCPCB in-stock selection verified 2026-09-22 -> JLCPCB sourcing selection verified 2026-09-25
- TP2, TP3, TP4: Assembly DNP - plated debug hole; no purchased component -> DNP - bare PCB test pad; no purchased component
