File: versions/v4.0-controller-serial-bridge/board.kicad_sch (KiCad schematic)
At the start: 80 parts, among them J1 J1 PS1 CONTROLLER - NOT USB, J2 J2 PS1 SERIAL - NOT USB, J3 J3 USB-C POWER / PROGRAM / PC, J5 AP63203WU-7, Q1 2N7002 DATA OPEN-DRAIN, Q2 2N7002 ACK OPEN-DRAIN, Q4 MMBT3904 AUTO RESET, Q5 MMBT3904 AUTO BOOT, SW1 RESET, SW2 BOOT, U1 ESP32-WROOM-32E, U2 CH340C, U4 AP2112K-3.3, U6 TPS2116DRLR POWER MUX

Commit message: Record JLC prototype order and synchronize V4.0 LED metadata
Parts:
- D8: LCSC C2286 -> C2986059; MPN 19-217/GHC-YR1S2/3T -> 19-217/GHC-YR1S2/6T
- D9: LCSC C2293 -> C2986058; MPN 19-217/BHC-ZL1M2RY/3T -> 19-217/BHC-ZL1M2RY/6T
Changed lines of the file:
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@@
 			)
 		)
-		(property "MPN" "19-217/GHC-YR1S2/3T"
+		(property "MPN" "19-217/GHC-YR1S2/6T"
 			(at 66.04 635 0)
 			(hide yes)
@@
 			)
 		)
-		(property "LCSC" "C2286"
+		(property "LCSC" "C2986059"
 			(at 66.04 635 0)
 			(hide yes)
@@
 			)
 		)
-		(property "MPN" "19-217/BHC-ZL1M2RY/3T"
+		(property "MPN" "19-217/BHC-ZL1M2RY/6T"
 			(at 101.6 635 0)
 			(hide yes)
@@
 			)
 		)
-		(property "LCSC" "C2293"
+		(property "LCSC" "C2986058"
 			(at 101.6 635 0)
 			(hide yes)
